File: electronics/KiCad/1_Distribution_Board/1_Distribution_Board.kicad_pcb (KiCad board)
At the start: 2 copper layers, 130 x 130 mm, 117 parts, among them J101 Conn_01x10, J102 Conn_01x06, J201 Jumper Pins, J202 Jumper Pins, J203 JST PH, J204 Generic 2.54mm, J301 Conn_01x02, J302 Conn_01x02, J401 Conn_01x02, J402 Conn_01x02, J5 Conn_01x04, J501 JST VH, J502 JST VH, J503 Barrel_Jack, J504 Barrel_Jack, J505 Conn_01x04, J601 Generic 2.54mm, J602 Generic 2.54mm, J603 Generic 2.54mm, J604 Generic 2.54mm, J605 Generic 2.54mm, J606 Generic 2.54mm, J701 Jumper Pins, J702 Jumper Pins, J703 JST PH, J704 Generic 2.54mm, J801 Jumper Pins, J802 Jumper Pins, J803 JST PH, J804 Generic 2.54mm, Q101 DMG2305UX, Q601 TBD, Q602 TBD, U501 LM7805_TO220, U502 LM317_TO-220, U503 LM7812_TO220

Commit message: Cleaned up Power
Updated power area to include RECOM only and adding stack flex cable connector as an in-case-of
Parts:
- removed A2 (x3): TMC2209_SILENTSTEPSTICK, TMC2209_SILENTSTEPSTICK:MODULE_TMC2209_SILENTSTEPSTICK
- removed J5: Conn_01x04, Connector_JST:JST_XA_B04B-XASK-1-A_1x04_P2.50mm_Vertical
- removed the REF** at (90.0, 90.0)
- removed the REF** at (90.0, 30.0)
- removed U501: LM7805_TO220, Package_TO_SOT_THT:TO-220-3_Vertical
- removed U502: LM317_TO-220, Package_TO_SOT_THT:TO-220-3_Vertical
- removed U503: LM7812_TO220, Package_TO_SOT_THT:TO-220-3_Vertical
- added A201: TMC2209_SILENTSTEPSTICK, TMC2209_SILENTSTEPSTICK:MODULE_TMC2209_SILENTSTEPSTICK, F.Cu at (126.0, 43.0)
- added A701: TMC2209_SILENTSTEPSTICK, TMC2209_SILENTSTEPSTICK:MODULE_TMC2209_SILENTSTEPSTICK, F.Cu at (124.0, 65.0)
- added A801: TMC2209_SILENTSTEPSTICK, TMC2209_SILENTSTEPSTICK:MODULE_TMC2209_SILENTSTEPSTICK, F.Cu at (124.0, 87.0)
- added C1: 10uf, Capacitor_SMD:C_0805_2012Metric_Pad1.18x1.45mm_HandSolder, F.Cu at (-27.0, 1.00)
- added C2: 10uf, Capacitor_SMD:C_0805_2012Metric_Pad1.18x1.45mm_HandSolder, F.Cu at (-27.0, 4.01)
- added C3: 10uf, Capacitor_SMD:C_0805_2012Metric_Pad1.18x1.45mm_HandSolder, F.Cu at (-27.0, 7.03)
- added C4: 10uf, Capacitor_SMD:C_0805_2012Metric_Pad1.18x1.45mm_HandSolder, F.Cu at (-27.0, 10.0)
- added C5: 10uf, Capacitor_SMD:C_0805_2012Metric_Pad1.18x1.45mm_HandSolder, F.Cu at (-27.0, 13.0)
- added C501: 10uf, Capacitor_SMD:C_0805_2012Metric_Pad1.18x1.45mm_HandSolder, F.Cu at (-27.0, 16.1)
- added D101: MBR120VLSFT1G, PCM_SparkFun-Semiconductor-Standard:SOD-123, F.Cu at (111.0, 31.0)
- added J506: JST VH, Connector_JST:JST_VH_B2P-VH-FB-B_1x02_P3.96mm_Vertical, F.Cu at (246.2, 40.9)
- added J507: JST VH, Connector_JST:JST_VH_B2P-VH-FB-B_1x02_P3.96mm_Vertical, F.Cu at (246.2, 52.6)
- added J508: JST VH, Connector_JST:JST_VH_B2P-VH-FB-B_1x02_P3.96mm_Vertical, F.Cu at (246.2, 64.4)
- added J509: JST VH, Connector_JST:JST_VH_B2P-VH-FB-B_1x02_P3.96mm_Vertical, F.Cu at (246.2, 76.2)
- added SW101: SW_Push, Button_Switch_THT:SW_PUSH_6mm, F.Cu at (106.3, 37.8)
- added U504: R-78C5.0-1.0, Converter_DCDC:Converter_DCDC_RECOM_R-78E-0.5_THT, F.Cu at (89.6, -35.8)
- added U505: R-786.5-0.5, Converter_DCDC:Converter_DCDC_RECOM_R-78E-0.5_THT, F.Cu at (89.6, -25.7)
- added U506: R-78B12-2.0, Converter_DCDC:Converter_DCDC_RECOM_R-78B-2.0_THT, F.Cu at (89.5, -19.9)
- moved F301 44.0 mm to (52.0, 135.5), turned to 180 degrees
- moved F401 39.1 mm to (106.0, 137.5), turned to 180 degrees
- moved DIAG_201 39.0 mm to (147.0, 46.1), turned to -90 degrees
- moved R101 33.2 mm to (106.0, 52.0), turned to -90 degrees
- moved J302 32.5 mm to (60.7, 146.5), turned to 90 degrees
- moved J202 30.4 mm to (160.0, 52.5)
- moved R206 28.3 mm to (142.5, 44.0), turned to -90 degrees
- moved R207 28.2 mm to (142.5, 48.0), turned to -90 degrees
- moved C301 28.1 mm to (50.3, 143.5)
- moved J201 25.7 mm to (160.0, 39.5)
- moved J401 25.4 mm to (127.3, 146.5), turned to -90 degrees
- moved J402 24.4 mm to (114.7, 146.5), turned to 90 degrees
- moved C401 22.6 mm to (104.0, 145.5)
- moved A301 21.1 mm to (75.4, 126.7)
- moved J301 19.9 mm to (71.8, 147.0), turned to -90 degrees
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Connections:
- net +7.5V renamed +6.5V
- net Net-(A102-PWM_0) renamed /PWM_0
- net Net-(A102-PWM_1) renamed /PWM_1
- net Net-(A102-PWM_2) renamed /PWM_2
- net Net-(A102-PWM_3) renamed /PWM_3
- net Net-(A102-PWM_4) renamed /PWM_4
- net Net-(A102-PWM_5) renamed /PWM_5
- net Net-(A102-PWM_6) renamed /PWM_6
- net Net-(A102-PWM_7) renamed /PWM_7
- net Net-(A102-PWM_8) renamed /PWM_8
- net Net-(A102-PWM_9) renamed /PWM_9

Commit message: Added 4th stepper
Added 4th stepper on SCH and PCB
Parts:
- added A8: TMC2209_SILENTSTEPSTICK, TMC2209_SILENTSTEPSTICK:MODULE_TMC2209_SILENTSTEPSTICK, F.Cu at (152.4, -34.2)
- added C16: 100uF, Capacitor_THT:CP_Radial_D8.0mm_P2.50mm, F.Cu at (169.3, -40.3)
- added DIAG_4: PTH, Connector_PinHeader_2.54mm:PinHeader_1x01_P2.54mm_Vertical, F.Cu at (167.9, -23.6)
- added INDX_4: PTH, Connector_PinHeader_2.54mm:PinHeader_1x01_P2.54mm_Vertical, F.Cu at (167.9, -19.0)
- added J35: Jumper Pins, Connector_PinHeader_2.54mm:PinHeader_1x03_P2.54mm_Vertical, F.Cu at (167.9, -33.2)
- added J36: Jumper Pins, Connector_PinHeader_2.54mm:PinHeader_1x03_P2.54mm_Vertical, F.Cu at (172.4, -33.2)
- added J37: JST PH, Connector_JST:JST_PH_B4B-PH-K_1x04_P2.00mm_Vertical, F.Cu at (146.5, -20.5)
- added J38: Generic 2.54mm, Connector_PinHeader_2.54mm:PinHeader_1x04_P2.54mm_Vertical, F.Cu at (172.4, -23.6)
- added PDN_4: PTH, Connector_PinHeader_2.54mm:PinHeader_1x01_P2.54mm_Vertical, F.Cu at (167.9, -14.4)
- added R43: 10k, Resistor_SMD:R_0805_2012Metric_Pad1.20x1.40mm_HandSolder, F.Cu at (163.2, -43.6)
- added R44: 10k, Resistor_SMD:R_0805_2012Metric_Pad1.20x1.40mm_HandSolder, F.Cu at (163.2, -40.7)
- added R45: 10k, Resistor_SMD:R_0805_2012Metric_Pad1.20x1.40mm_HandSolder, F.Cu at (163.2, -37.7)
- added R46: 10k, Resistor_SMD:R_0805_2012Metric_Pad1.20x1.40mm_HandSolder, F.Cu at (163.2, -34.8)
- added R47: 10k, Resistor_SMD:R_0805_2012Metric_Pad1.20x1.40mm_HandSolder, F.Cu at (163.2, -31.8)
- added R48: 10k, Resistor_SMD:R_0805_2012Metric_Pad1.20x1.40mm_HandSolder, F.Cu at (163.2, -28.9)
- added R49: 10k, Resistor_SMD:R_0805_2012Metric_Pad1.20x1.40mm_HandSolder, F.Cu at (163.2, -25.9)
- added R50: 10k, Resistor_SMD:R_0805_2012Metric_Pad1.20x1.40mm_HandSolder, F.Cu at (163.2, -23.0)
- added R51: 10k, Resistor_SMD:R_0805_2012Metric_Pad1.20x1.40mm_HandSolder, F.Cu at (163.2, -20.0)
- renumbered A101 to A1, A102 to A2, A201 to A3, A301 to A4, A401 to A5, A701 to A6, A801 to A7, C201 to C1, C601 to C10, C602 to C11, C603 to C12, C604 to C13, C701 to C14, C801 to C15, C301 to C2, C401 to C3, C501 to C4, C2 to C5, C4 to C6, C1 to C7, C3 to C8, C5 to C9, D101 to D1, DIAG_201 to DIAG_1, DIAG_701 to DIAG_2, DIAG_801 to DIAG_3, F301 to F1, F401 to F2, INDX_201 to INDX_1, INDX_701 to INDX_2, INDX_801 to INDX_3, J401 to J10, J402 to J11, J501 to J12, J504 to J13, J506 to J14, J507 to J15, J505 to J16, J502 to J17, J508 to J18, J509 to J19, J101 to J2, J503 to J20, J601 to J21, J603 to J22, J605 to J23, J606 to J24, J602 to J25, J604 to J26, J701 to J27, J702 to J28, J703 to J29, J102 to J3, J704 to J30, J801 to J31, J802 to J32, J803 to J33, J804 to J34, J201 to J4, J202 to J5, J203 to J6, J204 to J7, J301 to J8, J302 to J9, PDN_201 to PDN_1, PDN_701 to PDN_2, PDN_801 to PDN_3, Q101 to Q1, Q601 to Q2, Q602 to Q3, R102 to R1, R201 to R10, R206 to R11, R207 to R12, R601 to R13, R605 to R14, R609 to R15, R611 to R16, R602 to R17, R606 to R18, R610 to R19, R101 to R2, R612 to R20, R603 to R21, R607 to R22, R604 to R23, R608 to R24, R702 to R25, R704 to R26, R709 to R27, R703 to R28, R705 to R29, R103 to R3, R708 to R30, R701 to R31, R706 to R32, R707 to R33, R802 to R34, R804 to R35, R809 to R36, R803 to R37, R805 to R38, R808 to R39, R202 to R4, R801 to R40, R806 to R41, R807 to R42, R204 to R5, R209 to R6, R203 to R7, R205 to R8, R208 to R9, SW101 to SW1, U505 to U1, U506 to U2, U504 to U3

Commit message: Updated Layout
More positioning Layout
Parts:
- removed the REF** at (210.0, 90.0)
- removed the REF** at (30.0, 30.0)
- removed the REF** at (150.0, 30.0)
- removed the REF** at (150.0, 150.0)
- removed the REF** at (210.0, 150.0)
- removed the REF** at (30.0, 150.0)
- removed the REF** at (150.0, 90.0)
- removed the REF** at (30.0, 90.0)
- removed the REF** at (90.0, 150.0)
- removed the REF** at (210.0, 30.0)
- added M1: MountingHole_3.2mm_M3_ISO7380_Pad, MountingHole:MountingHole_3.2mm_M3_ISO7380_Pad, F.Cu at (150.0, 150.0)
- added M1: MountingHole_3.2mm_M3_ISO7380_Pad, MountingHole:MountingHole_3.2mm_M3_ISO7380_Pad, F.Cu at (30.0, 150.0)
- added M1: MountingHole_3.2mm_M3_ISO7380_Pad, MountingHole:MountingHole_3.2mm_M3_ISO7380_Pad, F.Cu at (30.0, 30.0)
- added M1: MountingHole_3.2mm_M3_ISO7380_Pad, MountingHole:MountingHole_3.2mm_M3_ISO7380_Pad, F.Cu at (150.2, 30.0)
- added M1: MountingHole_3.2mm_M3_ISO7380_Pad, MountingHole:MountingHole_3.2mm_M3_ISO7380_Pad, F.Cu at (90.0, 150.0)
- added M1: MountingHole_3.2mm_M3_ISO7380_Pad, MountingHole:MountingHole_3.2mm_M3_ISO7380_Pad, F.Cu at (150.0, 90.0)
- added M1: MountingHole_3.2mm_M3_ISO7380_Pad, MountingHole:MountingHole_3.2mm_M3_ISO7380_Pad, F.Cu at (30.0, 90.0)
- added REF**: PinHeader_1x02_P1.27mm_Vertical, Connector_PinHeader_1.27mm:PinHeader_1x02_P1.27mm_Vertical, F.Cu at (173.0, 40.0)
- added REF**: PinSocket_1x08_P2.54mm_Vertical, Connector_PinSocket_2.54mm:PinSocket_1x08_P2.54mm_Vertical, F.Cu at (193.0, 33.0)
- moved A8 169.0 mm to (130.0, 133.3), turned to 180 degrees
- moved C16 166.4 mm to (143.0, 124.0), turned to -90 degrees
- moved J38 160.0 mm to (147.0, 134.4)
- moved U2 155.3 mm to (105.8, 134.5), turned to 90 degrees
- moved J19 154.4 mm to (109.0, 147.0)
- moved J37 152.6 mm to (152.6, 132.0), turned to -90 degrees
- moved DIAG_4 150.6 mm to (122.4, 120.0)
- moved INDX_4 143.3 mm to (133.0, 120.0)
- moved U1 126.4 mm to (54.4, 95.8), turned to 180 degrees
- moved U3 121.6 mm to (88.4, 85.8), turned to 180 degrees
- moved R5 103.7 mm to (250.8, 100.8), turned to 0 degrees
- moved R6 103.0 mm to (71.0, 29.5), turned to -90 degrees
- moved J4 102.1 mm to (241.5, 101.0), turned to 90 degrees
- moved R4 94.2 mm to (236.0, 100.8), turned to 0 degrees
- moved R8 78.0 mm to (228.2, 101.2), turned to 0 degrees
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Other:
- board text added: "0"
- board text added: "0 mm"
- board text added: "0.0000 mm / 0.0000 mm"
- board text added: "0.01 mm"
- board text added: "0.02"
- board text added: "0.035 mm"
- board text added: "0.3000 mm"
- board text added: "1"
- board text added: "1 2 3"
- board text added: "1-2"
- board text added: "1.51 mm"
- board text added: "1.6000 mm"
- board text added: "1_Distribution_Board Assembly REV"
- board text added: "1_Distribution_Board PCB REV 0.1"
- board text added: "2"
- board text added: "2-3"
- board text added: "3.3"
- board text added: "4.5"
- board text added: "70.0000 mm x 50.0000 mm"
- board text added: "B.Cu"
- board text added: "B.Mask"
- board text added: "B.Paste"
- board text added: "B.Silkscreen"
- board text added: "BOARD CHARACTERISTICS"
- board text added: "Board Thickness:"
- board text added: "Board overall dimensions:"
- board text added: "Bottom Silk Screen"
- board text added: "Bottom Solder Mask"
- board text added: "Bottom Solder Paste"
- board text added: "Castellated pads:"
- board text added: "Color"
- board text added: "Copper Finish:"
- board text added: "Copper Layer Count:"
- board text added: "DIAG, pull high, pull low"
- board text added: "Dielectric 1"
- board text added: "Edge card connectors:"
- board text added: "Epsilon R"
- board text added: "F.Cu"
- board text added: "F.Mask"
- board text added: "F.Paste"
- board text added: "F.Silkscreen"
- board text added: "FR4"
- board text added: "FR4 natural"
- board text added: "Fix RX-TX Tie-in to only be one resistor"
- board text added: "Green"
- board text added: "HAL SnPb"
- board text added: "Impedance Control:"
- board text added: "JP4"
- board text added: "JP5"
- board text added: "Layer Name"
- board text added: "Loss Tangent"
- board text added: "MS1"
- board text added: "MS2"
- board text added: "Material"
- board text added: "Min hole diameter:"
- board text added: "Min track/spacing:"
- board text added: "No"
- board text added: "Not specified"
- board text added: "Plated Board Edge:"
- board text added: "Thickness (mm)"
- board text added: "Top Silk Screen"
- board text added: "Top Solder Mask"
- board text added: "Top Solder Paste"
- board text added: "Type"
- board text added: "White"
- board text added: "copper"
- board text added: "core"
- board text added: "~{EN} needs to only have one pull up?"

Commit message: Updated Schematic naming, PCB work
Updated Schematic naming for sub-sheets to get rid of untitled and adapter board ones. ADD - 815 sub-sheet for cleaner printable schematic.

PCB:

Started moving modules to socket headers for easy of prototyping.
Parts:
- removed A2: 815, 815:MODULE_815
- removed J2: Conn_01x10, Connector_JST:JST_XA_B10B-XASK-1-A_1x10_P2.50mm_Vertical
- removed J3: Conn_01x06, Connector_PinHeader_2.54mm:PinHeader_1x06_P2.54mm_Vertical
- removed R10, R27, R31, R36, R40, R45: 10k, Resistor_SMD:R_0805_2012Metric_Pad1.20x1.40mm_HandSolder
- removed REF**: PinHeader_1x02_P1.27mm_Vertical, Connector_PinHeader_1.27mm:PinHeader_1x02_P1.27mm_Vertical
- removed REF**: PinSocket_1x08_P2.54mm_Vertical, Connector_PinSocket_2.54mm:PinSocket_1x08_P2.54mm_Vertical
- added J1: Conn_02x08_Odd_Even, Connector_IDC:IDC-Header_2x08_P2.54mm_Vertical, F.Cu at (65.4, 139.0)
- added J40: Module Right, Connector_PinSocket_2.54mm:PinSocket_1x06_P2.54mm_Vertical, F.Cu at (32.9, 108.7)
- added J42: Signals 0-3, Connector_PinSocket_2.54mm:PinSocket_1x04_P2.54mm_Vertical, F.Cu at (38.0, 121.4)
- added J43: Signals 4-7, Connector_PinSocket_2.54mm:PinSocket_1x04_P2.54mm_Vertical, F.Cu at (50.7, 121.4)
- added J44: Signals 8-11, Connector_PinSocket_2.54mm:PinSocket_1x04_P2.54mm_Vertical, F.Cu at (65.9, 121.4)
- added J45: Conn_01x10, Connector_JST:JST_XA_B10B-XASK-1-A_1x10_P2.50mm_Vertical, F.Cu at (32.0, 140.0)
- added J46: Conn_01x06, Connector_PinHeader_2.54mm:PinHeader_1x06_P2.54mm_Vertical, F.Cu at (95.0, 142.5)
- added J47: Signals 12-15, Connector_PinSocket_2.54mm:PinSocket_1x04_P2.54mm_Vertical, F.Cu at (78.6, 121.4)
- added J48: Module Left, Connector_PinSocket_2.54mm:PinSocket_1x06_P2.54mm_Vertical, F.Cu at (91.2, 108.7)
- moved R49 310.7 mm to (-138.0, 50.2)
- moved R6 209.8 mm to (-138.0, 47.2), turned to 0 degrees
- moved R43 186.8 mm to (219.3, 134.6)
- moved R44 186.8 mm to (219.3, 137.5)
- moved R46 186.8 mm to (219.3, 143.4)
- moved R48 186.8 mm to (219.3, 149.3)
- moved R51 186.8 mm to (219.3, 158.2)
- moved J35 186.8 mm to (224.0, 144.9)
- moved J36 186.8 mm to (228.6, 144.9)
- moved R47 186.8 mm to (219.3, 146.3)
- moved R50 186.8 mm to (219.3, 155.2)
- moved PDN_4 186.8 mm to (224.0, 163.8)
- moved J10 162.2 mm to (-57.0, 88.0), turned to 180 degrees
- moved A5 158.6 mm to (-50.1, 66.7)
- moved C3 157.0 mm to (-76.0, 90.5)
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Connections:
- R6 pad 1: /UART0_TX -> /UART0_RX
- R6 pad 2: /UART0_RX -> /UART0_TX
Other:
- board text added: "A2"
