File: electronics/KiCad/1_Distribution_Board/815.kicad_sch (KiCad schematic)
At the start: 47 parts, among them J12 Conn_01x06, J13 Conn_01x10, J14 2.54-1*4P母, J15 2.54-1*4P母, J16 PM254V-11-06-H85, J17 Conn_02x08_Odd_Even, J18 PM254V-11-06-H85, J19 2.54-1*4P母, J20 2.54-1*4P母, U6 PCA9306, U7 PCA9685PW, Y1 25MHz

Commit message: Updated P/DNP for parts that should not be there for end users
Updated P/DNP for initial build to be sent out to additional people for sorter builds.
Parts:
- J14, J15, J16, J18, J19, J20: now not fitted
Changed lines of the file:
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@@
 		(in_bom yes)
 		(on_board yes)
-		(dnp no)
+		(dnp yes)
 		(fields_autoplaced yes)
 		(property "Reference" "J14"
@@
 		(in_bom yes)
 		(on_board yes)
-		(dnp no)
+		(dnp yes)
 		(fields_autoplaced yes)
 		(property "Reference" "J16"
@@
 		(in_bom yes)
 		(on_board yes)
-		(dnp no)
+		(dnp yes)
 		(fields_autoplaced yes)
 		(property "Reference" "J20"
@@
 		(in_bom yes)
 		(on_board yes)
-		(dnp no)
+		(dnp yes)
 		(fields_autoplaced yes)
 		(property "Reference" "J15"
@@
 		(in_bom yes)
 		(on_board yes)
-		(dnp no)
+		(dnp yes)
 		(fields_autoplaced yes)
 		(property "Reference" "J18"
@@
 		(in_bom yes)
 		(on_board yes)
-		(dnp no)
+		(dnp yes)
 		(fields_autoplaced yes)
 		(property "Reference" "J19"
