File: electronics/KiCad/1_Distribution_Board/815.kicad_sch (KiCad schematic)
At the start: 41 parts, among them J12 Conn_01x06, J13 Conn_01x10, J17 Conn_02x08_Odd_Even, U6 PCA9306, U7 PCA9685PW, Y1 25MHz

Commit message: distribution board v1.4: s1 on the silkscreen, ground stitching, small cleanups
Small fixes from a review of the v1.4 layout:

- The RESET button's reference, S1, is now printed on the top silkscreen,
  upright and left of the button, as proposed in #953. It is at least
  1.5 mm from every pad and clear of the RESET label. An assembly order
  was flagged earlier for the missing S1 marking.
- Y1 loses the PROD_ID field "XTAL-25500" left over from the SparkFun
  symbol, in the schematic and on the board. Its MPN, manufacturer, LCSC
  number and datasheet stay.
- The bottom-layer +3V3 strap to driver A4's MS2 pin (P7.3) now runs at
  y = 88.9 mm instead of 88.7 mm. It cleared the GND pin P7.2 by 0.21 mm;
  it now clears it by 0.41 mm.
- Removed a 0.12 mm VSYS track stub that lay entirely inside Y1 pad 1.
- Removed an unused copy of the old outline-only logo from User.Drawings,
  outside the board outline, so plotting that layer no longer prints it.
- The VSYS link that ran down the top layer under the logo is re-routed
  around its left side: the bottom-layer run continues at 45 degrees to
  y = 84 mm and left to a via at (83.5, 84.0), then a 0.5 mm top-layer
  track runs down x = 83.5 mm to the existing VSYS track at y = 97.32 mm.
  The ground pour under the logo is now one unbroken piece, with no
  clearance channels showing through the white silkscreen. The new path
  is about as long as the old one.
- Seven 0.6/0.3 mm GND vias stitch ground pour patches that joined the
  rest of ground at a single point, left where the jumper fields and the
  module headers were removed: two beside P1 pin 2 on the bottom layer,
  one beside P7 pin 2 on the bottom layer, one beside P13 pins 2 and 3 on
  the top layer, and one at the top end of each of the three top-layer
  ground strips between the PWM tracks below R55-R58.

DRC (zones refilled, all severities, schematic parity) shows the same
items as before and no unconnected items. ERC is unchanged. The netlist
is unchanged apart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
Parts:
- Y1: PROD_ID XTAL-25500 -> (none)
Changed lines of the file:
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@@
-			)
-		)
-		(property "PROD_ID" "XTAL-25500"
-			(at 59.69 133.35 0)
-			(hide yes)
-			(show_name no)
-			(do_not_autoplace no)
-			(effects
-				(font
-					(size 1.27 1.27)
-				)
 			)
 		)
