File: electronics/KiCad/1_Distribution_Board/Level_Shifters.kicad_sch (KiCad schematic)
At the start: 32 parts, among them J10 Generic 2.54mm, J11 Generic 2.54mm, J5 Generic 2.54mm, J6 Generic 2.54mm, J8 Generic 2.54mm, J9 Generic 2.54mm, Q2 AO3400A, Q3 AO3400A, Q4 AO3400A, Q5 AO3400A

Commit message: Fix Y1 oscillator supply routing and switch to 5V
Parts:
- JP1, JP2, JP3, JP4: value ~ -> (none)
