File: electronics/KiCad/1_Distribution_Board/Stepper_Module.kicad_sch (KiCad schematic)
At the start: 14 parts, among them J21 Jumper Pins, J22 Jumper Pins, J23 JST PH, J24 Generic 2.54mm, P1 Header-Female-2.54_1x8, P2 Header-Female-2.54_1x2, P3 Header-Female-2.54_1x8

Commit message: distribution board v1.4: hardwired driver addresses, led ports on 24 v, no module headers, fill-only logo, rev in silkscreen
Stepper driver UART addresses are now fixed in copper:
- Removed the ten MS1/MS2 jumper headers (J21, J22, J25, J26, J29, J30,
  J33, J34, J37, J38) and the twenty 10k resistors that served only them
  (R61-R64, R67-R70, R73-R76, R79-R82, R85-R88). The DIAG pull-ups R13,
  R16, R65, R66 and R71 stay, and so does R72, the series resistor of
  the VSYS LED D7.
- Each driver's MS1 (AD0) and MS2 (AD1) pins are tied straight to GND or
  +3V3 through new sheet pins on the root sheet: A2 = 0, A3 = 1, A4 = 2,
  A5 = 3 on UART0 and A6 = 0 on UART1. This is the address map the
  firmware already uses (TMC_UART_ADDRESSES), so firmware does not change.
- On the board the low pins join the ground pour, two of them through a
  short ground stitch and via, and the high pins get short bottom-layer
  +3V3 tracks. Tracks and vias that only served the jumpers are removed.
- Removed the jumper silkscreen: the Pins/Setting legend, the "1 2 3" and
  "3 2 1" pin numbers, the MS1/MS2 labels and "!Double check!".
- The Stepper_Module sheet loses its jumper block and microstep table; a
  note on the root sheet gives the address map.

LED and fan ports run straight from 24 V:
- Removed the 180 ohm resistors R21, R22, R27, R28 and the bypass solder
  jumpers JP1-JP4. Pin 1 of J8, J9, J10 and J11 now connects directly to
  +24V, the state v1.3 boards were built in with the bypasses bridged.
- Removed the four "Bypass Rxx" labels.

Plug-in PCA9685 module headers removed:
- Removed J14, J15, J16, J18, J19 and J20, the module's silkscreen outline,
  the "A10" label and the three tracks that only went to J16. A new ground
  via replaces J16's ground pin as the stitch for that patch of ground pour.
- The on-board PCA9685 (U7) and everything it uses stay, including the
  220 ohm output resistors R43-R58 on the path to J17 and J12.

Oscillator follow-ups:
- D1 (MBR120VLSFT1G, LC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
Parts:
- removed J21, J22: Jumper Pins, Connector_PinHeader_2.54mm:PinHeader_1x03_P2.54mm_Vertical, symbol Connector_Generic:Conn_01x03
- removed R61, R62, R63, R64: 10kΩ, PCM_JLCPCB:R_0603, symbol PCM_JLCPCB-Resistors:0603,10kΩ
Connections:
- no-connect marks 3 -> 4
Other:
- note added: "1k from RX to TX on MCU necessary for single wire UART"
- note added: "UART address, set on root sheet"
- note removed: "10k from RX to TX on MCU necessary for single wire UART"
- note removed: "Jumper Pins allow for configuration High or Low on MS1 and MS2 by simply adding a jumper across pins 1-2 or 2-3"
- note removed: "MS1 MS2 Steps Interpolation GND GND 8 Yes to 256 VIO GND 2 Yes to 256 GND VIO 4 Yes to 256 VIO VIO 16 Yes to 256"
- note removed: "Micro Step Setting"
- note removed: "Requires 2 Jumpers JLCPCB # C5305"
- note removed: "See Micro Step Setting"
