File: electronics/KiCad/1_Distribution_Board/Pi_Link.kicad_sch (KiCad schematic)
At the start: 7 parts, among them J41 2x9 socket, 15 mm (hand-fit), U8 ISO7721DR, U9 LTV-357T-C

Commit message: distribution board v1.5: j41 is a samtec esw-109-33-g-d
J41 names its part: a 2x9 elevated socket strip with a 16.13 mm body. On the
20 mm standoffs the Orange Pi 5 header pins go about 4.6 mm into it, inside
Samtec's 3.68 to 6.35 mm insertion range, and the socket stops about 1.4 mm
above the header's plastic. Still fitted by hand. ERC, DRC and schematic
parity unchanged.

Co-Authored-By: Claude Opus 5.5 <noreply@anthropic.com>
Parts:
- J41: value 2x9 socket, 15 mm (hand-fit) -> ESW-109-33-G-D (hand-fit); Notes Under the board, onto the Orange Pi 5 pins 1-18. Hand-fit: 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 -> Under the board, onto the Orange Pi 5 pins 1-18. Samtec ESW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
Changed lines of the file:
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@@
 			)
 		)
-		(property "Value" "2x9 socket, 15 mm (hand-fit)"
+		(property "Value" "ESW-109-33-G-D (hand-fit)"
 			(at 53.34 102.87 0)
 			(effects
@@
 			)
 		)
-		(property "Datasheet" ""
+		(property "Datasheet" "https://suddendocs.samtec.com/catalog_english/esw_th.pdf"
 			(at 60.96 88.9 0)
 			(hide yes)
@@
 			)
 		)
-		(property "Notes" "Under the board, onto the Orange Pi 5 pins 1-18. Hand-fit: 15 mm body for the 20 mm stack."
+		(property "Notes" "Under the board, onto the Orange Pi 5 pins 1-18. Samtec ESW-109-33-G-D: a 16.13 mm body, so on 20 mm standoffs the Pi's pins go about 4.6 mm in (Samtec: 3.68 to 6.35 mm). Fitted by hand."
 			(at 60.96 88.9 0)
 			(hide yes)

Commit message: distribution board v1.5: servo supply blocking diode, servo bus and pi-side test access
- D11 (SS34, LCSC C8678) in series from the servo regulator U5
  (R-78B6.5-1.5) to CN2 pin 2. This is RECOM's recommended "optional
  protection 2" for the R-78B: the servos' capacitance and back-driven
  motors can no longer push current into U5's output while U5 is off,
  and U5's capacitive-load limit rises from 1000 uF to 6800 uF. The
  connector side is the new net SERVO_PWR. Servos see about 0.4 V less,
  about 6.1 V at 1.5 A.
- J42, a not-fitted 2.54 mm pair just right of the serial servo
  connector (pin 1 SERVO_DATA, pin 2 GND), for a scope or logic analyser
  on the half-duplex servo bus while a servo is plugged in.
- TP_GND_PI_1, a test pad on GND_PI inside the isolated Pi island, as
  the probe ground on the Pi side of the UART isolator.
- Silkscreen: the board name and revision move right for J42, A6 moves
  below D11, Q2's reference steps off D11's outline, and J8's reference
  is hidden like J9's and J10's.

DRC with refilled zones: no errors, nothing unconnected, warnings as
before (16 silk overlaps, 5 courtyard overlaps; library notes 113 with
the three new footprints); parity reports only the JAW logo. ERC: the
same 3 errors carried from v1.4. JLC: the BOM adds D11 (basic part);
the CPL adds D11 at 90 degrees, which lands on JLC's own SMA footprint
for C8678 within 0.2 mm, cathode on pad 1.

Co-Authored-By: Claude Opus 5.5 <noreply@anthropic.com>
Parts:
- added TP_GND_PI_1: PTH, TestPoint:TestPoint_THTPad_D2.0mm_Drill1.0mm, symbol PCM_SparkFun-Connector:TestPoint_PTH
Connections:
- net GND_PI: now also TP_GND_PI_1.1
Changed lines of the file:
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@@
+		)
+	)
+	(symbol
+		(lib_id "PCM_SparkFun-Connector:TestPoint_PTH")
+		(at 55.88 50.8 0)
+		(unit 1)
+		(body_style 1)
+		(exclude_from_sim no)
+		(in_bom no)
+		(on_board yes)
+		(in_pos_files yes)
+		(dnp no)
+		(property "Reference" "TP_GND_PI_1"
+			(at 55.88 45.72 0)
+			(effects
+				(font
+					(size 1.27 1.27)
+				)
+				(justify left)
+			)
+		)
+		(property "Value" "PTH"
+			(at 58.42 52.07 0)
+			(effects
+				(font
+					(size 1.27 1.27)
+				)
+				(justify left)
+			)
+		)
+		(property "Footprint" "TestPoint:TestPoint_THTPad_D2.0mm_Drill1.0mm"
+			(at 55.88 50.8 0)
+			(hide yes)
+			(effects
+				(font
+					(size 1.27 1.27)
+				)
+			)
+		)
+		(property "Datasheet" ""
+			(at 55.88 50.8 0)
+			(hide yes)
+			(effects
+				(font
+					(size 1.27 1.27)
+				)
+			)
+		)
+		(property "Description" ""
+			(at 55.88 50.8 0)
+			(hide yes)
+			(effects
+				(font
+					(size 1.27 1.27)
+				)
+			)
+		)
+		(pin "1"
+		)
+		(instances
+			(project "1_Distribution_Board"
+				(path "/d53c8c01-e754-4310-8a73-7d7c95e64cd3/82c0cf1b-d902-4f9c-a05a-257f324ec865"
+					(reference "TP_GND_PI_1")
+					(unit 1)
+				)
+			)
+		)
+	)
+	(wire
+		(pts
+			(xy 55.88 50.8) (xy 55.88 53.339999999999996)
+		)
+		(stroke
+			(width 0)
+			(type default)
+		)
+	)
+	(label "GND_PI"
+		(at 55.88 53.339999999999996 270)
+		(effects
+			(font
+				(size 1.27 1.27)
+			)
+			(justify right bottom)
 		)
 	)

Commit message: distribution board v1.5: LED port clamps, GP7 pull-up, low-ESR bulk caps
- D12-D15 (BAS316) from each LED port's switched side to +24V, so an
  inductive load (a fan, a long lead) cannot push the 30 V AO3400A
  switches past their rating at turn-off. A silicon diode rather than a
  Schottky: these sit at 24 V reverse whenever their port is on, and a
  small Schottky's leakage can heat it into thermal runaway. BAS316 is
  rated 30 uA at 25 V with a 150 C junction.
- R105 (10k) pulls GP7, the Pico's TX to the Pi through the isolator, up
  to 3.3 V. The RP2040 holds its pins low through reset, which reached
  the Pi's RX as a break.
- C11-C15 become Panasonic EEE-FT1V101AP (0.26 ohm ESR and 300 mA ripple
  at 100 kHz) on the same footprint; the previous part gave no ESR.
- The isolated ground island ends 0.25 mm sooner, so the Pi side keeps
  1 mm from the board's copper (it was 0.88 mm at J36), with one via to
  keep the island's front fill joined.
- GP19 under U8 moves to the back layer so U8's ground pin stays joined
  to the pour.
- D11-D15 silkscreen lines are 0.15 mm.

Co-Authored-By: Claude Opus 5.5 <noreply@anthropic.com>
Parts:
- added R105: 10kΩ, PCM_JLCPCB:R_0603, symbol PCM_JLCPCB-Resistors:0603,10kΩ
Connections:
- net +3V3: now also R105.1
- net PICO_TX: now also R105.2
Changed lines of the file:
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@@
-		)
-	)
-	(wire
-		(pts
-			(xy 137.16 78.74) (xy 152.4 78.74)
-		)
-		(stroke
-			(width 0)
-			(type default)
 		)
 	)
@@
 		)
 	)
+	(wire
+		(pts
+			(xy 137.16 78.74) (xy 147.32 78.74)
+		)
+		(stroke
+			(width 0)
+			(type default)
+		)
+	)
+	(wire
+		(pts
+			(xy 147.32 78.74) (xy 152.4 78.74)
+		)
+		(stroke
+			(width 0)
+			(type default)
+		)
+	)
+	(junction
+		(at 147.32 78.74)
+		(diameter 0)
+		(color 0 0 0 0)
+	)
+	(symbol
+		(lib_id "PCM_JLCPCB-Resistors:0603,10kΩ")
+		(at 147.32 74.93 0)
+		(unit 1)
+		(body_style 1)
+		(exclude_from_sim no)
+		(in_bom yes)
+		(on_board yes)
+		(in_pos_files yes)
+		(dnp no)
+		(property "Reference" "R105"
+			(at 149.85999999999999 74.295 0)
+			(effects
+				(font
+					(size 1.27 1.27)
+				)
+				(justify left)
+			)
+		)
+		(property "Value" "10kΩ"
+			(at 149.85999999999999 76.83500000000001 0)
+			(effects
+				(font
+					(size 1.27 1.27)
+				)
+				(justify left)
+			)
+		)
+		(property "Footprint" "PCM_JLCPCB:R_0603"
+			(at 147.32 74.93 0)
+			(hide yes)
+			(effects
+				(font
+					(size 1.27 1.27)
+				)
+			)
+		)
+		(property "Datasheet" ""
+			(at 147.32 74.93 0)
+			(hide yes)
+			(effects
+				(font
+					(size 1.27 1.27)
+				)
+			)
+		)
+		(property "Description" ""
+			(at 147.32 74.93 0)
+			(hide yes)
+			(effects
+				(font
+					(size 1.27 1.27)
+				)
+			)
+		)
+		(property "LCSC" "C25804"
+			(at 147.32 74.93 0)
+			(hide yes)
+			(effects
+				(font
+					(size 1.27 1.27)
+				)
+			)
+		)
+		(property "Notes" "Holds GP7 (U8 INA) high while the Pico is in reset."
+			(at 147.32 74.93 0)
+			(hide yes)
+			(effects
+				(font
+					(size 1.27 1.27)
+				)
+			)
+		)
+		(pin "1"
+		)
+		(pin "2"
+		)
+		(instances
+			(project "1_Distribution_Board"
+				(path "/d53c8c01-e754-4310-8a73-7d7c95e64cd3/82c0cf1b-d902-4f9c-a05a-257f324ec865"
+					(reference "R105")
+					(unit 1)
+				)
+			)
+		)
+	)
+	(symbol
+		(lib_id "power:+3V3")
+		(at 147.32 71.12 0)
+		(unit 1)
+		(body_style 1)
+		(exclude_from_sim no)
+		(in_bom yes)
+		(on_board yes)
+		(in_pos_files yes)
+		(dnp no)
+		(property "Reference" "#PWR0337"
+			(at 149.85999999999999 69.85000000000001 0)
+			(hide yes)
+			(effects
+				(font
+					(size 1.27 1.27)
+				)
+				(justify left)
+			)
+		)
+		(property "Value" "+3V3"
+			(at 147.32 67.31 0)
+			(effects
+				(font
+					(size 1.27 1.27)
+				)
+				(justify left)
+			)
+		)
+		(property "Footprint" ""
+			(at 147.32 71.12 0)
+			(hide yes)
+			(effects
+				(font
+					(size 1.27 1.27)
+				)
+			)
+		)
+		(property "Datasheet" ""
+			(at 147.32 71.12 0)
+			(hide yes)
+			(effects
+				(font
+					(size 1.27 1.27)
+				)
+			)
+		)
+		(property "Description" ""
+			(at 147.32 71.12 0)
+			(hide yes)
+			(effects
+				(font
+					(size 1.27 1.27)
+				)
+			)
+		)
+		(instances
+			(project "1_Distribution_Board"
+				(path "/d53c8c01-e754-4310-8a73-7d7c95e64cd3/82c0cf1b-d902-4f9c-a05a-257f324ec865"
+					(reference "#PWR0337")
+					(unit 1)
+				)
+			)
+		)
+	)
